File: basic_stm32_board.kicad_sch (KiCad schematic)
At the start: 61 parts, among them J1 Screw_Terminal_01x02, J2 USB_B_Micro, J3 Conn_01x04, J4 Conn_01x04, J5 Conn_ARM_JTAG_SWD_10, Q1 AO3401A, SW1 SW_SPDT, U1 STM32F405RGT6, U2 MP2303ADN, U3 USBLC6-2SC6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

Commit message: changed some footprints
Parts:
- FB1: footprint Inductor_SMD:L_6.3x6.3_H3 -> Inductor_SMD:L_1206_3216Metric_Pad1.22x1.90mm_HandSolder
- L1: footprint Inductor_SMD:L_0402_1005Metric_Pad0.77x0.64mm_HandSolder -> Inductor_SMD:L_0603_1608Metric_Pad1.05x0.95mm_HandSolder
Changed lines of the file:
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@@
 			)
 		)
-		(property "Footprint" "Inductor_SMD:L_6.3x6.3_H3"
+		(property "Footprint" "Inductor_SMD:L_1206_3216Metric_Pad1.22x1.90mm_HandSolder"
 			(at 58.42 42.418 90)
 			(effects
@@
 			)
 		)
-		(property "Footprint" "Inductor_SMD:L_0402_1005Metric_Pad0.77x0.64mm_HandSolder"
+		(property "Footprint" "Inductor_SMD:L_0603_1608Metric_Pad1.05x0.95mm_HandSolder"
 			(at 93.98 77.47 0)
 			(effects
